Commit message: Fixed Gazebo Simulation

File: sdrc_description/urdf/mobile_base.xacro (robot description, xacro)
@@ -22,5 +22,5 @@
     <xacro:macro name="create_wheel_and_joint" params="prefix x y">
         <xacro:wheel_link prefix="${prefix}"/>
-        <joint name="base_${prefix}_wheel" type="continuous">
+        <joint name="base_${prefix}_wheel_joint" type="continuous">
             <parent link="base_link"/>
             <child link="${prefix}_wheel_link"/>

File: sdrc_description/urdf/mobile_base_gazebo.xacro (robot description, xacro)
@@ -22,5 +22,5 @@
         <material>Gazebo/Grey</material>
     </gazebo>
-    <gazebo>
+    <!-- <gazebo>
         <plugin name="object_controller" filename="libgazebo_ros_planar_move.so">
         <commandTopic>cmd_vel</commandTopic>
@@ -30,4 +30,35 @@
         <robotBaseFrame>base_footprint</robotBaseFrame>
         </plugin>
+    </gazebo> -->
+    <gazebo>
+        <plugin name="diff_drive_controller" filename="libgazebo_ros_diff_drive.so">
+            <!-- Update rate in Hz -->
+            <update_rate>50</update_rate>
+            <!-- wheels -->
+            <!-- Number of wheel pairs -->
+            <num_wheel_pairs>3</num_wheel_pairs>
+            <!-- wheels0 -->
+            <left_joint>base_left_front_wheel_joint</left_joint>
+            <right_joint>base_right_front_wheel_joint</right_joint>
+            <!-- wheels1-->
+            <left_joint>base_left_back_wheel_joint</left_joint>
+            <right_joint>base_right_back_wheel_joint</right_joint>
+            <left_joint>base_left_middle_wheel_joint</left_joint>
+            <right_joint>base_right_middle_wheel_joint</right_joint>
+            <!-- kinematics -->
+            <wheel_separation>0.5</wheel_separation>
+            <wheel_separation>0.5</wheel_separation>
+            <wheel_separation>0.5</wheel_separation>
+            <wheel_diameter>${wheel_radius} * 2</wheel_diameter>
+            <wheel_diameter>${wheel_radius} * 2</wheel_diameter>
+            <wheel_diameter>${wheel_radius} * 2</wheel_diameter>
+            <!-- output -->
+            <publish_odom>true</publish_odom>
+            <publish_odom_tf>true</publish_odom_tf>
+            <publish_wheel_tf>true</publish_wheel_tf>
+            <odometry_topic>odom</odometry_topic>
+            <odometry_frame>odom</odometry_frame>
+            <robot_base_frame>base_footprint</robot_base_frame>
+        </plugin>
     </gazebo>
 </robot>
