Commit message: feat(lidar): added lidar to simulation

File: sdrc_description/urdf/common_properties.xacro (robot description, xacro)
@@ -7,4 +7,7 @@
     <material name="grey">
         <color rgba="0.5 0.5 0.5 1" />
+    </material>
+    <material name="red">
+        <color rgba="1 0 0 1" />
     </material>
     <!-- Inertias -->

File: sdrc_description/urdf/constants.xacro (robot description, xacro)
@@ -1,4 +1,5 @@
 <?xml version="1.0"?>
 <robot xmlns:xacro="http://www.ros.org/wiki/xacro">
+    <!-- Chasis & Wheels -->
     <xacro:property name="base_length" value="0.6"/>
     <xacro:property name="base_width" value="0.4"/>
@@ -11,3 +12,7 @@
     <xacro:property name="chasis_weight_kgs" value="25" />
     <xacro:property name="wheel_weight_kgs" value="2" />
+    <!-- LiDar -->
+    <xacro:property name="lidar_radius" value="0.075"/>
+    <xacro:property name="lidar_length" value="0.05"/>
+    <xacro:property name="lidar_mass" value="0.1"/>
 </robot>

File: sdrc_description/urdf/my_robot.urdf.xacro (robot description, xacro)
@@ -5,3 +5,4 @@
     <xacro:include filename="mobile_base.xacro" />
     <xacro:include filename="mobile_base_gazebo.xacro" />
+    <xacro:include filename="lidar.xacro" />
 </robot>

Commit message: Integrated SLAM

File: sdrc_description/urdf/common_properties.xacro (robot description, xacro)
@@ -26,7 +26,5 @@
             <origin xyz="${xyz}" rpy="${rpy}" />
             <mass value="${m}" />
-            <inertia ixx="${(m/12) * (3*r*r + h*h)}" ixy="0" ixz="0"
-                     iyy="${(m/12) * (3*r*r + h*h)}" iyz="0"
-                     izz="${(m/2) * (r*r)}"/>
+            <inertia ixx="${(m/12) * (3*r*r + h*h)}" ixy = "0" ixz = "0" iyy="${(m/12) * (3*r*r + h*h)}" iyz = "0" izz="${(m/2) * (r*r)}"/>
         </inertial>
     </xacro:macro>

File: sdrc_description/urdf/constants.xacro (robot description, xacro)
@@ -10,9 +10,11 @@
     <xacro:property name="wheel_offset_y" value="${base_width / 2.0 + wheel_length / 2.0}" />
     <xacro:property name="base_origin_z" value="${base_height / 2.0}" />
+    <xacro:property name="axle_eff_limit" value="5.12766"/>
+    <xacro:property name="axle_vel_limit" value="244.8696"/>
     <xacro:property name="chasis_weight_kgs" value="5" />
-    <xacro:property name="wheel_weight_kgs" value="2" />
+    <xacro:property name="wheel_weight_kgs" value="0.5" />
     <!-- LiDar -->
-    <xacro:property name="lidar_radius" value="0.075"/>
-    <xacro:property name="lidar_length" value="0.05"/>
+    <xacro:property name="lidar_radius" value="0.05"/>
+    <xacro:property name="lidar_length" value="0.04"/>
     <xacro:property name="lidar_mass" value="0.1"/>
     <!-- Camera -->

File: sdrc_description/urdf/depth_camera.xacro (robot description, xacro)
@@ -2,5 +2,5 @@
 <robot xmlns:xacro="http://www.ros.org/wiki/xacro">
     <joint name="camera_joint" type="fixed">
-        <parent link="base_link"/>
+        <parent link="chassis"/>
         <child link="camera_link"/>
         <origin xyz="${base_length / 2} 0 ${base_height / 2}" rpy="0 0 0"/>

File: sdrc_description/urdf/gazebo_control.xacro (robot description, xacro)
@@ -7,5 +7,5 @@
         <odometryFrame>odom</odometryFrame>
         <odometryRate>20.0</odometryRate>
-        <robotBaseFrame>base_footprint</robotBaseFrame>
+        <robotBaseFrame>base_link</robotBaseFrame>
         </plugin>
     </gazebo> -->
@@ -26,10 +26,8 @@
             <right_joint>base_right_middle_wheel_joint</right_joint>
             <!-- kinematics -->
-            <wheel_separation>${wheel_length}+${base_width}</wheel_separation>
-            <wheel_separation>${wheel_length}+${base_width}</wheel_separation>
-            <wheel_separation>${wheel_length}+${base_width}</wheel_separation>
-            <wheel_diameter>${wheel_radius} * 2</wheel_diameter>
-            <wheel_diameter>${wheel_radius} * 2</wheel_diameter>
-            <wheel_diameter>${wheel_radius} * 2</wheel_diameter>
+            <wheel_separation>${wheel_length + base_width}</wheel_separation>
+            <wheel_diameter>${wheel_radius * 2}</wheel_diameter>
+            <max_wheel_torque>200.0</max_wheel_torque>
+            <max_wheel_acceleration>1.0</max_wheel_acceleration>
             <!-- output -->
             <publish_odom>true</publish_odom>
@@ -38,5 +36,5 @@
             <odometry_topic>odom</odometry_topic>
             <odometry_frame>odom</odometry_frame>
-            <robot_base_frame>base_footprint</robot_base_frame>
+            <robot_base_frame>base_link</robot_base_frame>
         </plugin>
     </gazebo>

File: sdrc_description/urdf/lidar.xacro (robot description, xacro)
@@ -2,9 +2,9 @@
 <robot xmlns:xacro="http://www.ros.org/wiki/xacro">
     <joint name="lidar_joint" type="fixed">
-        <parent link="base_link"/>
-        <child link="lidar_frame"/>
+        <parent link="chassis"/>
+        <child link="laser_frame"/>
         <origin xyz="${base_length / 4} 0 ${base_height + lidar_length / 2}" rpy="0 0 0"/>
     </joint>
-    <link name="lidar_frame">
+    <link name="laser_frame">
         <visual>
             <geometry>
@@ -20,9 +20,9 @@
         <xacro:cylinder_inertia m="${lidar_mass}" r="${lidar_radius}" h="${lidar_length}" xyz="0 0 0" rpy="0 0 0"/>
     </link>
-    <gazebo reference="lidar_frame">
+    <gazebo reference="laser_frame">
         <material>Gazebo/Red</material>
         <sensor name="laser" type="ray">
             <pose> 0 0 0 0 0 0 </pose>
-            <visualize>true</visualize>
+            <visualize>false</visualize>
             <update_rate>10</update_rate>
             <ray>
@@ -37,4 +37,5 @@
                     <min>0.3</min>
                     <max>12</max>
+                    <resolution>0.01</resolution>
                 </range>
             </ray>
@@ -44,5 +45,5 @@
                 </ros>
                 <output_type>sensor_msgs/LaserScan</output_type>
-                <frame_name>lidar_frame</frame_name>
+                <frame_name>laser_frame</frame_name>
             </plugin>
         </sensor>

File: sdrc_description/urdf/mobile_base.xacro (robot description, xacro)
@@ -13,4 +13,5 @@
                 <geometry>
                     <cylinder radius="${wheel_radius}" length="${wheel_length}" />
+                    <!-- <sphere radius="${wheel_radius}" /> -->
                 </geometry>
                 <origin xyz="0 0 0" rpy="${pi/2.0} 0 0" />
@@ -22,8 +23,10 @@
         <xacro:wheel_link prefix="${prefix}"/>
         <joint name="base_${prefix}_wheel_joint" type="continuous">
-            <parent link="base_link"/>
+            <parent link="chassis"/>
             <child link="${prefix}_wheel_link"/>
             <origin xyz="${x} ${y} 0" rpy="0 0 0"/>
             <axis xyz="0 1 0" />
+            <!-- <limit effort="${axle_eff_limit}" velocity="${axle_vel_limit}"/>
+            <dynamics damping="0" friction="4.0" /> -->
         </joint>
     </xacro:macro>
@@ -34,5 +37,5 @@
     <xacro:create_wheel_and_joint prefix="left_front" x="${wheel_offset_x}" y="${wheel_offset_y}" />
     <xacro:create_wheel_and_joint prefix="right_front" x="${wheel_offset_x}" y="${-wheel_offset_y}" />
-    <link name="base_link">
+    <link name="chassis">
         <visual>
             <geometry>
@@ -50,9 +53,15 @@
         <xacro:box_inertia m="${chasis_weight_kgs}" l="${base_length}" w="${base_width}" h="${base_height}" xyz="0 0 ${base_origin_z}" rpy="0 0 0"/>
     </link>
-    <link name="base_footprint"></link>
-    <joint name="base_base_footprint" type="fixed">
-        <parent link="base_footprint"/>
-        <child link="base_link"/>
+    <link name="base_link"></link>
+    <joint name="base_base_link" type="fixed">
+        <parent link="base_link"/>
+        <child link="chassis"/>
         <origin xyz="0 0 ${wheel_radius}" rpy="0 0 0"/>
     </joint>
+    <joint name="base_footprint_joint" type="fixed">
+        <parent link="base_link"/>
+        <child link="base_footprint"/>
+        <origin xyz="0 0 0" rpy="0 0 0"/>
+    </joint>
+    <link name="base_footprint"></link>
 </robot>

File: sdrc_description/urdf/mobile_base_gazebo.xacro (robot description, xacro)
@@ -1,36 +1,36 @@
 <?xml version="1.0"?>
 <robot xmlns:xacro="http://www.ros.org/wiki/xacro">
-    <gazebo reference="base_link">
+    <gazebo reference="chassis">
         <material>Gazebo/Blue</material>
     </gazebo>
     <gazebo reference="left_back_wheel_link">
+        <mu1 value="7.0" />
+        <mu2 value="7.0" />
         <material>Gazebo/Grey</material>
-        <mu1 value="0.5"/>
-        <mu2 value="0.2"/>
     </gazebo>
     <gazebo reference="right_back_wheel_link">
+        <mu1 value="7.0" />
+        <mu2 value="7.0" />
         <material>Gazebo/Grey</material>
-        <mu1 value="0.5"/>
-        <mu2 value="0.2"/>
     </gazebo>
     <gazebo reference="left_middle_wheel_link">
+        <mu1 value="7.0" />
+        <mu2 value="7.0" />
         <material>Gazebo/Grey</material>
-        <mu1 value="0.5"/>
-        <mu2 value="0.2"/>
     </gazebo>
     <gazebo reference="right_middle_wheel_link">
+        <mu1 value="7.0" />
+        <mu2 value="7.0" />
         <material>Gazebo/Grey</material>
-        <mu1 value="0.5"/>
-        <mu2 value="0.2"/>
     </gazebo>
     <gazebo reference="left_front_wheel_link">
+        <mu1 value="7.0" />
+        <mu2 value="7.0" />
         <material>Gazebo/Grey</material>
-        <mu1 value="0.5"/>
-        <mu2 value="0.2"/>
     </gazebo>
     <gazebo reference="right_front_wheel_link">
+        <mu1 value="7.0" />
+        <mu2 value="7.0" />
         <material>Gazebo/Grey</material>
-        <mu1 value="0.5"/>
-        <mu2 value="0.2"/>
     </gazebo>
 </robot>

File: sdrc_description/urdf/my_robot.urdf.xacro (robot description, xacro)
@@ -13,4 +13,4 @@
     </xacro:unless>
     <xacro:include filename="lidar.xacro" />
-    <xacro:include filename="depth_camera.xacro" />
+    <!-- <xacro:include filename="depth_camera.xacro" /> -->
 </robot>
