Commit message: feat: added realistic mesh to simulation

File: sdrc_description/urdf/gazebo_control.xacro (robot description, xacro)
@@ -18,11 +18,11 @@
             <num_wheel_pairs>3</num_wheel_pairs>
             <!-- wheels0 -->
-            <left_joint>base_left_front_wheel_joint</left_joint>
-            <right_joint>base_right_front_wheel_joint</right_joint>
+            <left_joint>left_front_wheel_joint</left_joint>
+            <right_joint>right_front_wheel_joint</right_joint>
             <!-- wheels1-->
-            <left_joint>base_left_back_wheel_joint</left_joint>
-            <right_joint>base_right_back_wheel_joint</right_joint>
-            <left_joint>base_left_middle_wheel_joint</left_joint>
-            <right_joint>base_right_middle_wheel_joint</right_joint>
+            <left_joint>left_rear_wheel_joint</left_joint>
+            <right_joint>right_rear_wheel_joint</right_joint>
+            <left_joint>left_middle_wheel_joint</left_joint>
+            <right_joint>right_middle_wheel_joint</right_joint>
             <!-- kinematics -->
             <wheel_separation>${wheel_length + base_width}</wheel_separation>

File: sdrc_description/urdf/mobile_base_gazebo.xacro (robot description, xacro)
@@ -4,5 +4,5 @@
         <material>Gazebo/Blue</material>
     </gazebo>
-    <gazebo reference="left_back_wheel_link">
+    <gazebo reference="left_rear_wheel_link">
         <mu1 value="1.0"/>
         <mu2 value="0.7"/>
@@ -12,5 +12,5 @@
         <material>Gazebo/Grey</material>
     </gazebo>
-    <gazebo reference="right_back_wheel_link">
+    <gazebo reference="right_rear_wheel_link">
         <mu1 value="1.0"/>
         <mu2 value="0.7"/>

File: sdrc_description/urdf/my_robot.urdf.xacro (robot description, xacro)
@@ -2,8 +2,9 @@
 <robot name="my_robot" xmlns:xacro="http://www.ros.org/wiki/xacro">
     <xacro:arg name="use_ros2_control" default="true" />
-    <xacro:include filename="constants.xacro" />
+    <!-- <xacro:include filename="constants.xacro" />
     <xacro:include filename="common_properties.xacro" />
-    <xacro:include filename="mobile_base.xacro" />
-    <xacro:include filename="mobile_base_gazebo.xacro" />
+    <xacro:include filename="mobile_base.xacro" /> -->
+    <xacro:include filename="mesh_test_11.urdf.xacro" />
+    <!-- <xacro:include filename="mobile_base_gazebo.xacro" /> -->
     <xacro:if value="$(arg use_ros2_control)">
         <xacro:include filename="ros2_control.xacro" />
@@ -12,6 +13,6 @@
         <xacro:include filename="gazebo_control.xacro" />
     </xacro:unless>
-    <xacro:include filename="lidar.xacro" />
+    <!-- <xacro:include filename="lidar.xacro" />
     <xacro:include filename="gps.xacro" />
-    <xacro:include filename="depth_camera.xacro" />
+    <xacro:include filename="depth_camera.xacro" /> -->
 </robot>

File: sdrc_description/urdf/ros2_control.xacro (robot description, xacro)
@@ -5,5 +5,5 @@
             <plugin>gazebo_ros2_control/GazeboSystem</plugin>
         </hardware>
-        <joint name="base_left_front_wheel_joint">
+        <joint name="left_front_wheel_joint">
             <command_interface name="velocity">
                 <param name="min">-10</param>
@@ -13,5 +13,5 @@
             <state_interface name="position"/>
         </joint>
-        <joint name="base_left_middle_wheel_joint">
+        <joint name="left_middle_wheel_joint">
             <command_interface name="velocity">
                 <param name="min">-10</param>
@@ -21,5 +21,5 @@
             <state_interface name="position"/>
         </joint>
-        <joint name="base_left_back_wheel_joint">
+        <joint name="left_rear_wheel_joint">
             <command_interface name="velocity">
                 <param name="min">-10</param>
@@ -29,5 +29,5 @@
             <state_interface name="position"/>
         </joint>
-        <joint name="base_right_front_wheel_joint">
+        <joint name="right_front_wheel_joint">
             <command_interface name="velocity">
                 <param name="min">-10</param>
@@ -37,5 +37,5 @@
             <state_interface name="position"/>
         </joint>
-        <joint name="base_right_middle_wheel_joint">
+        <joint name="right_middle_wheel_joint">
             <command_interface name="velocity">
                 <param name="min">-10</param>
@@ -45,5 +45,5 @@
             <state_interface name="position"/>
         </joint>
-        <joint name="base_right_back_wheel_joint">
+        <joint name="right_rear_wheel_joint">
             <command_interface name="velocity">
                 <param name="min">-10</param>

Commit message: Fixed bug with ROS2 Control and URDf

File: sdrc_description/urdf/gazebo_control.xacro (robot description, xacro)
@@ -17,15 +17,16 @@
             <!-- Number of wheel pairs -->
             <num_wheel_pairs>3</num_wheel_pairs>
+            <!-- joints misnamed smh -->
             <!-- wheels0 -->
-            <left_joint>left_front_wheel_joint</left_joint>
-            <right_joint>right_front_wheel_joint</right_joint>
+            <left_joint>right_front_wheel_joint</left_joint>
+            <right_joint>left_front_wheel_joint</right_joint>
             <!-- wheels1-->
-            <left_joint>left_rear_wheel_joint</left_joint>
-            <right_joint>right_rear_wheel_joint</right_joint>
-            <left_joint>left_middle_wheel_joint</left_joint>
-            <right_joint>right_middle_wheel_joint</right_joint>
+            <left_joint>right_rear_wheel_joint</left_joint>
+            <right_joint>left_rear_wheel_joint</right_joint>
+            <left_joint>right_middle_wheel_joint</left_joint>
+            <right_joint>left_middle_wheel_joint</right_joint>
             <!-- kinematics -->
-            <wheel_separation>0.762</wheel_separation>
-            <wheel_diameter>0.2</wheel_diameter>
+            <!-- <wheel_separation>0.762</wheel_separation>
+            <wheel_diameter>0.2</wheel_diameter> -->
             <max_wheel_torque>200.0</max_wheel_torque>
             <max_wheel_acceleration>1.0</max_wheel_acceleration>

File: sdrc_description/urdf/robot_body.urdf.xacro (robot description, xacro)
@@ -52,5 +52,5 @@
         rpy="0 0 0" />
       <mass
-        value="0.48944" />
+        value="0.5" />
       <inertia
         ixx="0.0021898"
@@ -89,5 +89,5 @@
     type="fixed">
     <origin
-      xyz="-0.34589 0 -0.022225"
+      xyz="-0.35 0 -0.022"
       rpy="0 0 0" />
     <parent
@@ -105,12 +105,12 @@
         rpy="0 0 0" />
       <mass
-        value="1.38515667925253" />
-      <inertia
-        ixx="0.00608670649414915"
-        ixy="-1.51546150586869E-10"
-        ixz="5.01389386245008E-08"
-        iyy="0.00331734776435004"
-        iyz="1.79208088841883E-11"
-        izz="0.00331733123659271" />
+        value="1.39" />
+      <inertia
+        ixx="0.001"
+        ixy="0.000"
+        ixz="0.000"
+        iyy="0.001"
+        iyz="0.000"
+        izz="0.001" />
     </inertial>
     <visual>
@@ -136,4 +136,25 @@
           filename="package://sdrc_description/meshes/left_front_wheel_link.STL" />
       </geometry>
+      <surface>
+        <friction>
+          <ode>
+            <mu>100000.0</mu>
+            <mu2>100000.0</mu2>
+            <fdir1>0 0 0</fdir1>
+            <slip1>0.0</slip1>
+            <slip2>0.0</slip2>
+          </ode>
+          <contact>
+            <ode>
+              <soft_cfm>0</soft_cfm>
+              <soft_erp>0.2</soft_erp>
+              <kp>1e+5</kp>
+              <kd>1</kd>
+              <max_vel>0.01</max_vel>
+              <!-- <min_depth>0.001</min_depth> -->
+            </ode>
+          </contact>
+        </friction>
+      </surface>
     </collision>
   </link>
@@ -142,5 +163,5 @@
     type="continuous">
     <origin
-      xyz="-0.026131 -0.43501 -0.2454"
+      xyz="-0.026 -0.435 -0.245"
       rpy="0 0 0" />
     <parent
@@ -158,5 +179,5 @@
         rpy="0 0 0" />
       <mass
-        value="0.451855581637783" />
+        value="0.45" />
       <inertia
         ixx="0.000557359425591044"
@@ -195,5 +216,5 @@
     type="fixed">
     <origin
-      xyz="-0.0223501233974425 0.215899727447913 -0.0587375886680441"
+      xyz="-0.022 0.22 -0.059"
       rpy="0 0 0" />
     <parent
@@ -211,12 +232,12 @@
         rpy="0 0 0" />
       <mass
-        value="1.3852" />
-      <inertia
-        ixx="0.0060867"
-        ixy="-1.3047E-10"
-        ixz="5.0163E-08"
-        iyy="0.0033173"
-        iyz="5.842E-11"
-        izz="0.0033173" />
+        value="1.39" />
+      <inertia
+        ixx="0.001"
+        ixy="0.000"
+        ixz="0.000"
+        iyy="0.001"
+        iyz="0.000"
+        izz="0.001" />
     </inertial>
     <visual>
@@ -242,4 +263,25 @@
           filename="package://sdrc_description/meshes/left_rear_wheel_link.STL" />
       </geometry>
+      <surface>
+        <friction>
+          <ode>
+            <mu>100000.0</mu>
+            <mu2>100000.0</mu2>
+            <fdir1>0 0 0</fdir1>
+            <slip1>0.0</slip1>
+            <slip2>0.0</slip2>
+          </ode>
+        </friction>
+        <contact>
+            <ode>
+              <soft_cfm>0</soft_cfm>
+              <soft_erp>0.2</soft_erp>
+              <kp>1e+5</kp>
+              <kd>1</kd>
+              <max_vel>0.01</max_vel>
+              <!-- <min_depth>0.001</min_depth> -->
+            </ode>
+          </contact>
+      </surface>
     </collision>
   </link>
@@ -248,5 +290,5 @@
     type="continuous">
     <origin
-      xyz="-0.041844 0.21591 -0.18572"
+      xyz="-0.042 0.216 -0.193"
       rpy="0 0 0" />
     <parent
@@ -264,12 +306,12 @@
         rpy="0 0 0" />
       <mass
-        value="1.3852" />
-      <inertia
-        ixx="0.0060867"
-        ixy="3.7938E-08"
-        ixz="3.2773E-08"
-        iyy="0.0033173"
-        iyz="-8.2013E-09"
-        izz="0.0033173" />
+        value="1.39" />
+      <inertia
+        ixx="0.001"
+        ixy="0.000"
+        ixz="0.000"
+        iyy="0.001"
+        iyz="0.000"
+        izz="0.001" />
     </inertial>
     <visual>
@@ -295,4 +337,25 @@
           filename="package://sdrc_description/meshes/left_middle_wheel_link.STL" />
       </geometry>
+      <surface>
+        <friction>
+          <ode>
+            <mu>100000.0</mu>
+            <mu2>100000.0</mu2>
+            <fdir1>0 0 0</fdir1>
+            <slip1>0.0</slip1>
+            <slip2>0.0</slip2>
+          </ode>
+        </friction>
+        <contact>
+            <ode>
+              <soft_cfm>0</soft_cfm>
+              <soft_erp>0.2</soft_erp>
+              <kp>1e+5</kp>
+              <kd>1</kd>
+              <max_vel>0.01</max_vel>
+              <!-- <min_depth>0.001</min_depth> -->
+            </ode>
+          </contact>
+      </surface>
     </collision>
   </link>
@@ -301,5 +364,5 @@
     type="continuous">
     <origin
-      xyz="-0.041844 -0.21589 -0.18572"
+      xyz="-0.042 -0.22 -0.19"
       rpy="0 0 0" />
     <parent
@@ -317,5 +380,5 @@
         rpy="0 0 0" />
       <mass
-        value="0.49894" />
+        value="0.5" />
       <inertia
         ixx="0.0021898"
@@ -354,5 +417,5 @@
     type="fixed">
     <origin
-      xyz="0.346075000000017 0 -0.0222249999792783"
+      xyz="0.35 0 -0.022"
       rpy="0 0 0" />
     <parent
@@ -370,12 +433,12 @@
         rpy="0 0 0" />
       <mass
-        value="0.451855561191559" />
-      <inertia
-        ixx="0.000557359394151881"
-        ixy="-3.90638921000188E-08"
-        ixz="1.73581089366397E-07"
-        iyy="0.000207816780451024"
-        iyz="-1.29419748686903E-05"
-        izz="0.000444163205151771" />
+        value="0.45" />
+      <inertia
+        ixx="0.000557359425591044"
+        ixy="3.94579138177333E-08"
+        ixz="-1.73611323725284E-07"
+        iyy="0.000207816779409454"
+        iyz="-1.29419652457806E-05"
+        izz="0.000444163243659817" />
     </inertial>
     <visual>
@@ -407,5 +470,5 @@
     type="fixed">
     <origin
-      xyz="0.022224999999983 0.215899999971175 -0.0587375000128591"
+      xyz="0.022 0.22 -0.059"
       rpy="0 0 0" />
     <parent
@@ -423,12 +486,12 @@
         rpy="0 0 0" />
       <mass
-        value="1.38515667925641" />
-      <inertia
-        ixx="0.00608670649415985"
-        ixy="-3.81060675117107E-08"
-        ixz="-3.26231551854187E-08"
-        iyy="0.00331733827450242"
-        iyz="-8.43766950773987E-09"
-        izz="0.00331734072645102" />
+        value="1.39" />
+      <inertia
+        ixx="0.001"
+        ixy="0.000"
+        ixz="0.000"
+        iyy="0.001"
+        iyz="0.000"
+        izz="0.001" />
     </inertial>
     <visual>
@@ -454,4 +517,25 @@
           filename="package://sdrc_description/meshes/right_middle_wheel_link.STL" />
       </geometry>
+      <surface>
+        <friction>
+          <ode>
+            <mu>100000.0</mu>
+            <mu2>100000.0</mu2>
+            <fdir1>0 0 0</fdir1>
+            <slip1>0.0</slip1>
+            <slip2>0.0</slip2>
+          </ode>
+        </friction>
+        <contact>
+            <ode>
+              <soft_cfm>0</soft_cfm>
+              <soft_erp>0.2</soft_erp>
+              <kp>1e+5</kp>
+              <kd>1</kd>
+              <max_vel>0.01</max_vel>
+              <!-- <min_depth>0.001</min_depth> -->
+            </ode>
+          </contact>
+      </surface>
     </collision>
   </link>
@@ -460,5 +544,5 @@
     type="continuous">
     <origin
-      xyz="0.041863 -0.2159 -0.18574"
+      xyz="0.042 -0.22 -0.19"
       rpy="0 0 0" />
     <parent
@@ -476,12 +560,12 @@
         rpy="0 0 0" />
       <mass
-        value="1.38515667925022" />
-      <inertia
-        ixx="0.00608670649414288"
-        ixy="-1.51613486823585E-10"
-        ixz="-5.0138297667682E-08"
-        iyy="0.00331734776436555"
-        iyz="-1.68192191724776E-11"
-        izz="0.00331733123657076" />
+        value="1.39" />
+      <inertia
+        ixx="0.001"
+        ixy="0.000"
+        ixz="0.000"
+        iyy="0.001"
+        iyz="0.000"
+        izz="0.001" />
     </inertial>
     <visual>
@@ -507,4 +591,25 @@
           filename="package://sdrc_description/meshes/right_rear_wheel_link.STL" />
       </geometry>
+      <surface>
+        <friction>
+          <ode>
+            <mu>100000.0</mu>
+            <mu2>100000.0</mu2>
+            <fdir1>0 0 0</fdir1>
+            <slip1>0.0</slip1>
+            <slip2>0.0</slip2>
+          </ode>
+        </friction>
+        <contact>
+            <ode>
+              <soft_cfm>0</soft_cfm>
+              <soft_erp>0.2</soft_erp>
+              <kp>1e+5</kp>
+              <kd>1</kd>
+              <max_vel>0.01</max_vel>
+              <!-- <min_depth>0.001</min_depth> -->
+            </ode>
+          </contact>
+      </surface>
     </collision>
   </link>
@@ -513,5 +618,5 @@
     type="continuous">
     <origin
-      xyz="0.041863 0.2159 -0.18574"
+      xyz="0.042 0.216 -0.193"
       rpy="0 0 0" />
     <parent
@@ -529,12 +634,12 @@
         rpy="0 0 0" />
       <mass
-        value="1.38515666192677" />
-      <inertia
-        ixx="0.00608043301185015"
-        ixy="-0.000128488906642026"
-        ixz="2.8718884613149E-05"
-        iyy="0.00332332272916639"
-        iyz="-1.33545971335827E-06"
-        izz="0.00331762969863137" />
+        value="1.39" />
+      <inertia
+        ixx="0.001"
+        ixy="0.000"
+        ixz="0.000"
+        iyy="0.001"
+        iyz="0.000"
+        izz="0.001" />
     </inertial>
     <visual>
@@ -560,4 +665,25 @@
           filename="package://sdrc_description/meshes/right_front_wheel_link.STL" />
       </geometry>
+      <surface>
+        <friction>
+          <ode>
+            <mu>100000.0</mu>
+            <mu2>100000.0</mu2>
+            <fdir1>0 0 0</fdir1>
+            <slip1>0.0</slip1>
+            <slip2>0.0</slip2>
+          </ode>
+        </friction>
+        <contact>
+            <ode>
+              <soft_cfm>0</soft_cfm>
+              <soft_erp>0.2</soft_erp>
+              <kp>1e+5</kp>
+              <kd>1</kd>
+              <max_vel>0.01</max_vel>
+              <!-- <min_depth>0.001</min_depth> -->
+            </ode>
+          </contact>
+      </surface>
     </collision>
   </link>
@@ -566,5 +692,5 @@
     type="continuous">
     <origin
-      xyz="0.0259691526115853 -0.435038958244363 -0.245355896930363"
+      xyz="0.026 -0.435 -0.245"
       rpy="0 0 0" />
     <parent
@@ -576,14 +702,14 @@
   </joint>
   <link name="base_link"></link>
-    <joint name="base_base_link" type="fixed">
-        <parent link="base_link"/>
-        <child link="chassis"/>
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
File: sdrc_description/urdf/ros2_control.xacro (robot description, xacro)
@@ -56,4 +56,6 @@
     <gazebo>
         <plugin name="gazebo_ros2_control" filename="libgazebo_ros2_control.so">
+            <robot_param>robot_description</robot_param>
+            <robot_param_node>robot_state_publisher</robot_param_node>
             <parameters>$(find sdrc_description)/config/controllers.yaml</parameters>
         </plugin>
