Commit message: feat(world): Created a world with cones and obstacles to test autonomy, also integrated launch script to easily run simulation in enviornment

File: sdrc_description/urdf/constants.xacro (robot description, xacro)
@@ -5,5 +5,5 @@
     <xacro:property name="base_height" value="0.2"/>
     <xacro:property name="wheel_radius" value="0.1"/>
-    <xacro:property name="wheel_length" value="0.1"/>
+    <xacro:property name="wheel_length" value="0.05"/>
     <xacro:property name="wheel_offset_x" value="${base_length / 2.0}" />
     <xacro:property name="wheel_offset_y" value="${base_width / 2.0 + wheel_length / 2.0}" />

File: sdrc_description/urdf/mobile_base.xacro (robot description, xacro)
@@ -1,5 +1,4 @@
 <?xml version="1.0"?>
 <robot xmlns:xacro="http://www.ros.org/wiki/xacro">
-    <xacro:include filename="constants.xacro" />
     <xacro:macro name="wheel_link" params="prefix">
         <link name="${prefix}_wheel_link">

File: sdrc_description/urdf/mobile_base_gazebo.xacro (robot description, xacro)
@@ -47,7 +47,7 @@
             <right_joint>base_right_middle_wheel_joint</right_joint>
             <!-- kinematics -->
-            <wheel_separation>0.5</wheel_separation>
-            <wheel_separation>0.5</wheel_separation>
-            <wheel_separation>0.5</wheel_separation>
+            <wheel_separation>${wheel_length}+${base_width}</wheel_separation>
+            <wheel_separation>${wheel_length}+${base_width}</wheel_separation>
+            <wheel_separation>${wheel_length}+${base_width}</wheel_separation>
             <wheel_diameter>${wheel_radius} * 2</wheel_diameter>
             <wheel_diameter>${wheel_radius} * 2</wheel_diameter>

File: sdrc_description/urdf/my_robot.urdf.xacro (robot description, xacro)
@@ -1,4 +1,5 @@
 <?xml version="1.0"?>
 <robot name="my_robot" xmlns:xacro="http://www.ros.org/wiki/xacro">
+    <xacro:include filename="constants.xacro" />
     <xacro:include filename="common_properties.xacro" />
     <xacro:include filename="mobile_base.xacro" />

Commit message: feat(camera): added depth camera to simulation

File: sdrc_description/urdf/constants.xacro (robot description, xacro)
@@ -16,3 +16,7 @@
     <xacro:property name="lidar_length" value="0.05"/>
     <xacro:property name="lidar_mass" value="0.1"/>
+    <!-- Camera -->
+    <xacro:property name="camera_length" value="0.03"/>
+    <xacro:property name="camera_width" value="0.03"/>
+    <xacro:property name="camera_height" value="0.01"/>
 </robot>

File: sdrc_description/urdf/lidar.xacro (robot description, xacro)
@@ -4,5 +4,5 @@
         <parent link="base_link"/>
         <child link="lidar_frame"/>
-        <origin xyz="${- base_length / 4} 0 ${base_height + lidar_length / 2}" rpy="0 0 0"/>
+        <origin xyz="${base_length / 4} 0 ${base_height + lidar_length / 2}" rpy="0 0 0"/>
     </joint>
     <link name="lidar_frame">

File: sdrc_description/urdf/my_robot.urdf.xacro (robot description, xacro)
@@ -6,3 +6,4 @@
     <xacro:include filename="mobile_base_gazebo.xacro" />
     <xacro:include filename="lidar.xacro" />
+    <xacro:include filename="depth_camera.xacro" />
 </robot>

Commit message: feat(control): integrated ros2 control for the motors

File: sdrc_description/urdf/constants.xacro (robot description, xacro)
@@ -10,5 +10,5 @@
     <xacro:property name="wheel_offset_y" value="${base_width / 2.0 + wheel_length / 2.0}" />
     <xacro:property name="base_origin_z" value="${base_height / 2.0}" />
-    <xacro:property name="chasis_weight_kgs" value="25" />
+    <xacro:property name="chasis_weight_kgs" value="5" />
     <xacro:property name="wheel_weight_kgs" value="2" />
     <!-- LiDar -->

File: sdrc_description/urdf/mobile_base_gazebo.xacro (robot description, xacro)
@@ -6,59 +6,31 @@
     <gazebo reference="left_back_wheel_link">
         <material>Gazebo/Grey</material>
+        <mu1 value="0.5"/>
+        <mu2 value="0.2"/>
     </gazebo>
     <gazebo reference="right_back_wheel_link">
         <material>Gazebo/Grey</material>
+        <mu1 value="0.5"/>
+        <mu2 value="0.2"/>
     </gazebo>
     <gazebo reference="left_middle_wheel_link">
         <material>Gazebo/Grey</material>
+        <mu1 value="0.5"/>
+        <mu2 value="0.2"/>
     </gazebo>
     <gazebo reference="right_middle_wheel_link">
         <material>Gazebo/Grey</material>
+        <mu1 value="0.5"/>
+        <mu2 value="0.2"/>
     </gazebo>
     <gazebo reference="left_front_wheel_link">
         <material>Gazebo/Grey</material>
+        <mu1 value="0.5"/>
+        <mu2 value="0.2"/>
     </gazebo>
     <gazebo reference="right_front_wheel_link">
         <material>Gazebo/Grey</material>
-    </gazebo>
-    <!-- <gazebo>
-        <plugin name="object_controller" filename="libgazebo_ros_planar_move.so">
-        <commandTopic>cmd_vel</commandTopic>
-        <odometryTopic>odom</odometryTopic>
-        <odometryFrame>odom</odometryFrame>
-        <odometryRate>20.0</odometryRate>
-        <robotBaseFrame>base_footprint</robotBaseFrame>
-        </plugin>
-    </gazebo> -->
-    <gazebo>
-        <plugin name="diff_drive_controller" filename="libgazebo_ros_diff_drive.so">
-            <!-- Update rate in Hz -->
-            <update_rate>50</update_rate>
-            <!-- wheels -->
-            <!-- Number of wheel pairs -->
-            <num_wheel_pairs>3</num_wheel_pairs>
-            <!-- wheels0 -->
-            <left_joint>base_left_front_wheel_joint</left_joint>
-            <right_joint>base_right_front_wheel_joint</right_joint>
-            <!-- wheels1-->
-            <left_joint>base_left_back_wheel_joint</left_joint>
-            <right_joint>base_right_back_wheel_joint</right_joint>
-            <left_joint>base_left_middle_wheel_joint</left_joint>
-            <right_joint>base_right_middle_wheel_joint</right_joint>
-            <!-- kinematics -->
-            <wheel_separation>${wheel_length}+${base_width}</wheel_separation>
-            <wheel_separation>${wheel_length}+${base_width}</wheel_separation>
-            <wheel_separation>${wheel_length}+${base_width}</wheel_separation>
-            <wheel_diameter>${wheel_radius} * 2</wheel_diameter>
-            <wheel_diameter>${wheel_radius} * 2</wheel_diameter>
-            <wheel_diameter>${wheel_radius} * 2</wheel_diameter>
-            <!-- output -->
-            <publish_odom>true</publish_odom>
-            <publish_odom_tf>true</publish_odom_tf>
-            <publish_wheel_tf>true</publish_wheel_tf>
-            <odometry_topic>odom</odometry_topic>
-            <odometry_frame>odom</odometry_frame>
-            <robot_base_frame>base_footprint</robot_base_frame>
-        </plugin>
+        <mu1 value="0.5"/>
+        <mu2 value="0.2"/>
     </gazebo>
 </robot>

File: sdrc_description/urdf/my_robot.urdf.xacro (robot description, xacro)
@@ -5,4 +5,6 @@
     <xacro:include filename="mobile_base.xacro" />
     <xacro:include filename="mobile_base_gazebo.xacro" />
+    <!-- <xacro:include filename="gazebo_control.xacro" /> -->
+    <xacro:include filename="ros2_control.xacro" />
     <xacro:include filename="lidar.xacro" />
     <xacro:include filename="depth_camera.xacro" />

Commit message: fix: updated the code to use the meshes

File: sdrc_description/urdf/constants.xacro (robot description, xacro)
@@ -10,6 +10,4 @@
     <xacro:property name="wheel_offset_y" value="${base_width / 2.0 + wheel_length / 2.0}" />
     <xacro:property name="base_origin_z" value="${base_height / 2.0}" />
-    <xacro:property name="axle_eff_limit" value="5.12766"/>
-    <xacro:property name="axle_vel_limit" value="244.8696"/>
     <xacro:property name="chasis_weight_kgs" value="5" />
     <xacro:property name="wheel_weight_kgs" value="0.5" />

File: sdrc_description/urdf/my_robot.urdf.xacro (robot description, xacro)
@@ -5,5 +5,5 @@
     <xacro:include filename="common_properties.xacro" />
     <xacro:include filename="mobile_base.xacro" /> -->
-    <xacro:include filename="mesh_test_11.urdf.xacro" />
+    <xacro:include filename="robot_body.urdf.xacro" />
     <!-- <xacro:include filename="mobile_base_gazebo.xacro" /> -->
     <xacro:if value="$(arg use_ros2_control)">

Commit message: fix: added camera + gps to new model

File: sdrc_description/urdf/constants.xacro (robot description, xacro)
@@ -20,3 +20,5 @@
     <xacro:property name="camera_width" value="0.03"/>
     <xacro:property name="camera_height" value="0.01"/>
+    <xacro:property name="camera_y_location" value="-0.3"/>
+    <xacro:property name="camera_z_location" value="-0.1"/>
 </robot>

File: sdrc_description/urdf/depth_camera.xacro (robot description, xacro)
@@ -4,5 +4,5 @@
         <parent link="chassis"/>
         <child link="camera_link"/>
-        <origin xyz="${base_length / 2} 0 ${base_height / 2}" rpy="0 0 0"/>
+        <origin xyz="0 ${camera_y_location} ${camera_z_location}" rpy="0 0 ${ - pi / 2}"/>
     </joint>
     <link name="camera_link">

File: sdrc_description/urdf/my_robot.urdf.xacro (robot description, xacro)
@@ -2,7 +2,7 @@
 <robot name="my_robot" xmlns:xacro="http://www.ros.org/wiki/xacro">
     <xacro:arg name="use_ros2_control" default="true" />
-    <!-- <xacro:include filename="constants.xacro" />
+    <xacro:include filename="constants.xacro" />
     <xacro:include filename="common_properties.xacro" />
-    <xacro:include filename="mobile_base.xacro" /> -->
+    <!-- <xacro:include filename="mobile_base.xacro" />   -->
     <xacro:include filename="robot_body.urdf.xacro" />
     <!-- <xacro:include filename="mobile_base_gazebo.xacro" /> -->
@@ -13,6 +13,6 @@
         <xacro:include filename="gazebo_control.xacro" />
     </xacro:unless>
-    <!-- <xacro:include filename="lidar.xacro" />
+    <!-- <xacro:include filename="lidar.xacro" /> -->
     <xacro:include filename="gps.xacro" />
-    <xacro:include filename="depth_camera.xacro" /> -->
+    <xacro:include filename="depth_camera.xacro" />
 </robot>

Commit message: fixed a bug with map and odom transforms

File: sdrc_description/urdf/constants.xacro (robot description, xacro)
@@ -2,6 +2,6 @@
 <robot xmlns:xacro="http://www.ros.org/wiki/xacro">
     <!-- Chasis & Wheels -->
-    <xacro:property name="base_length" value="0.6"/>
-    <xacro:property name="base_width" value="0.4"/>
+    <xacro:property name="base_length" value="0.4"/>
+    <xacro:property name="base_width" value="0.6"/>
     <xacro:property name="base_height" value="0.2"/>
     <xacro:property name="wheel_radius" value="0.1"/>
@@ -20,5 +20,5 @@
     <xacro:property name="camera_width" value="0.03"/>
     <xacro:property name="camera_height" value="0.01"/>
-    <xacro:property name="camera_y_location" value="-0.3"/>
+    <xacro:property name="camera_x_location" value="0.3"/>
     <xacro:property name="camera_z_location" value="-0.1"/>
 </robot>

File: sdrc_description/urdf/depth_camera.xacro (robot description, xacro)
@@ -4,5 +4,5 @@
         <parent link="chassis"/>
         <child link="camera_link"/>
-        <origin xyz="0 ${camera_y_location} ${camera_z_location}" rpy="0 0 ${ - pi / 2}"/>
+        <origin xyz="${camera_x_location} 0 ${camera_z_location}" rpy="0 0 0"/>
     </joint>
     <link name="camera_link">

File: sdrc_description/urdf/gps.xacro (robot description, xacro)
@@ -16,5 +16,5 @@
     <joint name="gps_joint" type="fixed">
         <axis xyz="1 0 0"/>
-        <origin xyz="0 0 ${base_height}"/>
+        <origin xyz="0 0 ${base_height}" rpy="0 0 ${pi / 2}"/>
         <parent link="chassis"/>
         <child link="gps"/>

File: sdrc_description/urdf/robot_body.urdf.xacro (robot description, xacro)
@@ -24,5 +24,5 @@
       <origin
         xyz="0 0 0"
-        rpy="0 0 0" />
+        rpy="0 0 ${pi / 2}" />
       <geometry>
         <mesh
@@ -38,5 +38,5 @@
       <origin
         xyz="0 0 0"
-        rpy="0 0 0" />
+        rpy="0 0 ${pi / 2}" />
       <geometry>
         <mesh
@@ -50,5 +50,5 @@
       <origin
         xyz="0.015875 -0.13783 -0.047232"
-        rpy="0 0 0" />
+        rpy="0 0 ${pi / 2}" />
       <mass
         value="0.5" />
@@ -64,5 +64,5 @@
       <origin
         xyz="0 0 0"
-        rpy="0 0 0" />
+        rpy="0 0 ${pi / 2}" />
       <geometry>
         <mesh
@@ -78,5 +78,5 @@
       <origin
         xyz="0 0 0"
-        rpy="0 0 0" />
+        rpy="0 0 ${pi / 2}" />
       <geometry>
         <mesh
@@ -89,5 +89,5 @@
     type="fixed">
     <origin
-      xyz="-0.35 0 -0.022"
+      xyz="0 -0.35 -0.022"
       rpy="0 0 0" />
     <parent
@@ -163,6 +163,6 @@
     type="continuous">
     <origin
-      xyz="-0.026 -0.435 -0.245"
-      rpy="0 0 0" />
+      xyz="0.435 -0.026 -0.245"
+      rpy="0 0 ${pi / 2}" />
     <parent
       link="left_bogie_link" />
@@ -216,6 +216,6 @@
     type="fixed">
     <origin
-      xyz="-0.022 0.22 -0.059"
-      rpy="0 0 0" />
+      xyz="-0.22 -0.022 -0.059"
+      rpy="0 0 ${pi / 2}" />
     <parent
       link="left_bogie_link" />
@@ -378,5 +378,5 @@
       <origin
         xyz="0.015875 0.13783 -0.047232"
-        rpy="0 0 0" />
+        rpy="0 0 ${pi / 2}" />
       <mass
         value="0.5" />
@@ -392,5 +392,5 @@
       <origin
         xyz="0 0 0"
-        rpy="0 0 0" />
+        rpy="0 0 ${pi / 2}" />
       <geometry>
         <mesh
@@ -406,5 +406,5 @@
       <origin
         xyz="0 0 0"
-        rpy="0 0 0" />
+        rpy="0 0 ${pi / 2}" />
       <geometry>
         <mesh
@@ -417,5 +417,5 @@
     type="fixed">
     <origin
-      xyz="0.35 0 -0.022"
+      xyz="0 0.35 -0.022"
       rpy="0 0 0" />
     <parent
@@ -470,6 +470,6 @@
     type="fixed">
     <origin
-      xyz="0.022 0.22 -0.059"
-      rpy="0 0 0" />
+      xyz="-0.22 0.022 -0.059"
+      rpy="0 0 ${pi / 2}" />
     <parent
       link="right_bogie_link" />
@@ -692,6 +692,6 @@
     type="continuous">
     <origin
-      xyz="0.026 -0.435 -0.245"
-      rpy="0 0 0" />
+      xyz="0.435 0.026 -0.245"
+      rpy="0 0 ${pi / 2}" />
     <parent
       link="right_bogie_link" />
@@ -705,11 +705,5 @@
       <parent link="base_link"/>
       <child link="chassis"/>
-      <origin xyz="0 0 0.35" rpy="0 0 ${pi / 2}"/>
-  </joint>
-  <joint name="base_footprint_joint" type="fixed">
-      <parent link="base_link"/>
-      <child link="base_footprint"/>
-      <origin xyz="0 0 0" rpy="0 0 0"/>
-  </joint>
-  <link name="base_footprint"></link>
+      <origin xyz="0 0 0.35" rpy="0 0 0"/>
+  </joint>
 </robot>
