Commit message: added lidar + gps

File: sdrc_description/urdf/lidar.xacro (robot description, xacro)
@@ -4,5 +4,5 @@
         <parent link="chassis"/>
         <child link="laser_frame"/>
-        <origin xyz="${base_length / 4} 0 ${base_height + lidar_length / 2}" rpy="0 0 0"/>
+        <origin xyz="0 0 ${base_height + 0.25}" rpy="0 0 0"/>
     </joint>
     <link name="laser_frame">

File: sdrc_description/urdf/my_robot.urdf.xacro (robot description, xacro)
@@ -1,5 +1,5 @@
 <?xml version="1.0"?>
 <robot name="my_robot" xmlns:xacro="http://www.ros.org/wiki/xacro">
-    <xacro:arg name="use_ros2_control" default="true" />
+    <xacro:arg name="use_ros2_control" default="false" />
     <xacro:include filename="constants.xacro" />
     <xacro:include filename="common_properties.xacro" />
@@ -13,5 +13,5 @@
         <xacro:include filename="gazebo_control.xacro" />
     </xacro:unless>
-    <!-- <xacro:include filename="lidar.xacro" /> -->
+    <xacro:include filename="lidar.xacro" />
     <xacro:include filename="gps.xacro" />
     <xacro:include filename="depth_camera.xacro" />

Commit message: fixed a bug with local costmap and adjusted params to improve autonomous navigation

File: sdrc_description/urdf/lidar.xacro (robot description, xacro)
@@ -4,5 +4,5 @@
         <parent link="chassis"/>
         <child link="laser_frame"/>
-        <origin xyz="0 0 ${base_height + 0.25}" rpy="0 0 0"/>
+        <origin xyz="0 0 ${base_height + 0.2}" rpy="0 0 0"/>
     </joint>
     <link name="laser_frame">
