Commit message: New features for the autonomy side

File: sdrc_description/urdf/gps.xacro (robot description, xacro)
@@ -20,4 +20,11 @@
         <child link="gps"/>
     </joint>
+    <!-- Standard gps_link alias for downstream tools expecting this frame -->
+    <link name="gps_link"></link>
+    <joint name="gps_link_joint" type="fixed">
+        <parent link="gps"/>
+        <child link="gps_link"/>
+        <origin xyz="0 0 0" rpy="0 0 0"/>
+    </joint>
     <gazebo reference="gps">
         <sensor name="gps" type="gps">
@@ -27,5 +34,5 @@
                 <remapping>~/out:=data</remapping>
                 </ros>
-                <frame_name>gps</frame_name>
+                <frame_name>gps_link</frame_name>
             </plugin>
             <always_on>true</always_on>
